File: MD_Stable.kicad_pcb (KiCad board)
At the start: 2 copper layers, 100 x 100 mm, 308 parts, among them J1 Conn_02x04_Counter_Clockwise, J10 Conn_02x06_Odd_Even, J11 Conn_01x08_Pin, J12 Conn_01x05_Socket, J2 XT30_Male, J3 XT60_Male, J4 RE1, J5 RE2, J6 RE3, J7 MO_XT60_Female1, J8 MO_XT60_Female2, J9 MO_XT60_Female3, Q1 MTB7D0N6RJ3, Q10 MTB7D0N6RJ3, Q11 MTB7D0N6RJ3, Q12 MTB7D0N6RJ3, Q2 MTB7D0N6RJ3, Q3 MTB7D0N6RJ3, Q4 MTB7D0N6RJ3, Q5 MTB7D0N6RJ3, Q6 MTB7D0N6RJ3, Q7 MTB7D0N6RJ3, Q8 MTB7D0N6RJ3, Q9 MTB7D0N6RJ3, SW1 SW_Push, SW2 SW_Push, SW3 PWM, SW4 PWM, SW5 PWM, SW6 DIR, SW7 DIR, SW8 DIR, U1 NJM7808SDL1, U10 74AHC1G08W5, U11 74AHC1G08W5, U12 74AHC1G08W5, U13 IRS2302S, U14 IRS2302S, U15 IRS2302S, U16 NE555D, U17 IRS2302S, U18 IRS2302S, U19 IRS2302S, U2 BA05CC0Tに似た何か, U20 74AHC1G08W5, U21 74AHC1G08W5, U22 74AHC1G08W5, U23 UTRS485G-S08-R, U24 UTRS485G-S08-R, U3 STM32G431K8Tx, U4 BA05CC0Tに似た何か, U5 BA033CC0FP, U6 π160M60, U7 74AHC1G04W5, U8 74AHC1G04W5, U9 74AHC1G04W5

Commit message: 配線終わり見えてきた
Parts:
- added F1: Polyfuse, MyLib:PolyFuse_MF-NSMF-series, F.Cu at (130.8, 140.5)
- C7: moved to B.Cu
- C75: moved to F.Cu
- moved D50 29.2 mm to (197.2, 131.8), turned to 180 degrees
- moved D52 28.6 mm to (197.2, 105.2), turned to 180 degrees
- moved D53 27.2 mm to (197.2, 78.2), turned to 0 degrees
- moved R43 26.2 mm to (199.0, 130.3), turned to 0 degrees
- moved R44 25.6 mm to (199.0, 103.6), turned to 0 degrees
- moved D49 25.4 mm to (197.2, 128.8), turned to 0 degrees
- moved D51 24.7 mm to (197.2, 102.1), turned to 0 degrees
- moved R45 24.3 mm to (199.0, 76.7), turned to 0 degrees
- moved D54 23.4 mm to (197.2, 75.2), turned to 180 degrees
- moved R48 20.1 mm to (194.3, 80.7), turned to -90 degrees
- moved R50 19.8 mm to (194.2, 54.0), turned to -90 degrees
- moved R46 19.2 mm to (194.3, 107.9), turned to -90 degrees
- moved D45 17.4 mm to (192.3, 81.2), turned to 90 degrees
- moved D47 17.2 mm to (192.1, 54.5), turned to 90 degrees
- moved D59 16.9 mm to (193.8, 76.3), turned to -90 degrees
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Connections:
- C2 pad 1: +12V -> Net-(D4-K)
- D4 pad 1: +12V -> Net-(D4-K)
- J12 pad 1: Net-(J12-Pin_1) -> GNDD
- J12 pad 5: GNDD -> Net-(J12-Pin_5)
- J3 pad : (no net) -> GND
- J7 pad : (no net) -> GND
- J8 pad : (no net) -> GND
- J9 pad : (no net) -> GND
- R78 pad 1: Net-(J12-Pin_1) -> Net-(J12-Pin_2)
- R78 pad 2: Net-(J12-Pin_2) -> Net-(J12-Pin_3)
- R79 pad 1: Net-(J12-Pin_3) -> Net-(J12-Pin_4)
- R79 pad 2: Net-(J12-Pin_4) -> Net-(J12-Pin_5)
- R80 pad 1: Net-(J12-Pin_2) -> Net-(J12-Pin_3)
- R81 pad 2: Net-(J12-Pin_1) -> Net-(J12-Pin_2)
- R82 pad 1: Net-(J12-Pin_4) -> Net-(J12-Pin_5)
- R83 pad 2: Net-(J12-Pin_3) -> Net-(J12-Pin_4)
- U2 pad 1: +12V -> Net-(D4-K)
- U23 pad 6: Net-(J12-Pin_1) -> Net-(J12-Pin_2)
- U23 pad 7: Net-(J12-Pin_2) -> Net-(J12-Pin_3)
- U24 pad 6: Net-(J12-Pin_3) -> Net-(J12-Pin_4)
- U24 pad 7: Net-(J12-Pin_4) -> Net-(J12-Pin_5)
Routing:
- net GND: track 0.00 -> 596.3 mm, vias 0 -> 43
- net GNDD: track 103.2 -> 388.2 mm, vias 2 -> 24
- net VCC: track 0.00 -> 210.7 mm, vias 0 -> 6
- net +8V: track 0.00 -> 189.4 mm, vias 0 -> 1
- net +5V: track 0.00 -> 154.0 mm, vias 0 -> 2
- net +3V3: track 60.4 -> 208.8 mm
- net 555_Out_A: track 0.00 -> 126.3 mm
- net LED_1: track 2.44 -> 67.7 mm
- net Source_1A: track 0.00 -> 60.0 mm, vias 0 -> 6
- net Source_2A: track 0.00 -> 57.8 mm, vias 0 -> 224
- net Source_3A: track 0.00 -> 56.2 mm, vias 0 -> 6
- net +5VD: track 182.6 -> 227.9 mm, vias 4 -> 8
- net out_DIR3: track 0.00 -> 40.7 mm, vias 0 -> 3
- net Source_1B: track 0.00 -> 40.0 mm, vias 0 -> 6
- net Source_3B: track 0.00 -> 39.8 mm, vias 0 -> 6
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- added copper zone on B.Cu, net GND
- added copper zone on F.Cu, net GND
- added copper zone on B.Cu, net GNDD
- added copper zone on F.Cu, net GNDD
- added copper zone on B.Cu, net Source_1A
- added copper zone on F.Cu, net Source_1A
- added copper zone on B.Cu, net Source_1B
- added copper zone on F.Cu, net Source_1B
- added copper zone on B.Cu, net Source_2A
- added copper zone on F.Cu, net Source_2A
- added copper zone on B.Cu, net Source_2B
- added copper zone on F.Cu, net Source_2B
- added copper zone on B.Cu, net Source_3A
- added copper zone on F.Cu, net Source_3A
- added copper zone on B.Cu, net Source_3B
- added copper zone on F.Cu, net Source_3B
- added copper zone on F.Cu, net VCC

Commit message: MD基板完成
Parts:
- added G***: LOGO, MyLib:BDCrogidrive_nega, B.Cu at (123.4, 54.6)
- added ref**: val**, MyLib:ROGIKEN, F.Cu at (120.5, 98.3)
- moved R13 8.04 mm to (196.1, 134.6), turned to 90 degrees
- moved R14 1.95 mm to (110.7, 147.2)
- moved C5 1.22 mm to (120.8, 137.7), turned to 180 degrees
- moved D14 1.11 mm to (196.1, 138.1), turned to 90 degrees
- moved R77 0.86 mm to (146.9, 77.7)
- moved C52 0.77 mm to (189.4, 104.1)
- moved D57 0.77 mm to (193.8, 102.7)
- moved R57 0.77 mm to (191.8, 103.2)
- moved C45 0.74 mm to (189.4, 80.5)
- moved R48 0.74 mm to (194.3, 81.4)
- moved D45 0.74 mm to (192.3, 81.9)
- moved C4 0.70 mm to (164.7, 134.4)
- moved R27 0.60 mm to (146.7, 117.6)
- moved R76 0.60 mm to (146.9, 104.4)
- moved R29 0.56 mm to (147.2, 64.3)
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Routing:
- net GND: track 596.3 -> 876.0 mm, vias 43 -> 932
- net +5V: track 154.0 -> 150.8 mm
- net VCC: track 210.7 -> 208.1 mm, vias 6 -> 56
- net GNDD: track 388.2 -> 390.8 mm, vias 24 -> 448
- net DIR2: track 52.8 -> 54.8 mm
- net DIR1: track 61.4 -> 62.7 mm
- net +5VD: track 227.9 -> 226.7 mm
- net +8V: track 189.4 -> 190.5 mm
- net PWM1: track 59.8 -> 60.4 mm
- net Source_2A: vias 224 -> 234
- net Source_3B: vias 6 -> 230
- net Source_3A: vias 6 -> 223
- net Source_2B: vias 216 -> 230
- net Source_1B: vias 6 -> 235
- net Source_1A: vias 6 -> 226
- added copper zone on B.Cu, net VCC
Other:
- outline, holes or cut-outs redrawn
- board text added: "->RX:A"
- board text added: "->RX:B"
- board text added: "12V"
- board text added: "3V3"
- board text added: "8V"
- board text added: "<-TX:A"
- board text added: "<-TX:B"
- board text added: "A相"
- board text added: "B相"
- board text added: "DCMotor Driver Rev3.0 @KayOChef_meme"
- board text added: "DRIVE POWER"
- board text added: "ENC1"
- board text added: "ENC2"
- board text added: "ENC3"
- board text added: "LOGIC POWER"
- board text added: "MCO"
- board text added: "MO1"
- board text added: "MO2"
- board text added: "MO3"
- board text added: "NC"
- board text added: "RESET"
- board text added: "RX<-"
- board text added: "SWCLK"
- board text added: "SWDIO"
- board text added: "TIM2"
- board text added: "TIM3"
- board text added: "TIM4"
- board text added: "TX->"
- board text added: "USER PA7"
- board text added: "USER PB8"
- board text added: "VCC"
- board text removed: "5VA <-TX:A <-TX:B ->RX:A ->RX:B GND1"

Commit message: 製造番号位置指定
Other:
- board text added: "JLCJLCJLCJLC"
Changed lines of the file:
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@@
+		)
+	)
+	(gr_text "JLCJLCJLCJLC"
+		(at 200.406 121.158 90)
+		(layer "F.SilkS")
+		(effects
+			(font
+				(size 1 1)
+				(thickness 0.1)
+			)
+			(justify left bottom)
 		)
 	)

Commit message: rev3.1
Parts:
- removed the D43 at (192.3, 108.6)
- removed the D44 at (166.9, 116.1)
- removed the D45 at (192.3, 81.9)
- removed the D46 at (166.5, 89.7)
- removed the D47 at (192.1, 54.5)
- removed the D48 at (166.5, 62.7)
- removed the D55 at (193.8, 129.9)
- removed the D56 at (166.9, 129.5)
- removed the D57 at (193.8, 102.7)
- removed the D58 at (166.7, 102.9)
- removed the D59 at (193.8, 76.1)
- removed the D60 at (166.5, 76.2)
- removed the R45 at (199.0, 76.7)
- removed the R47 at (166.3, 118.1)
- removed the R49 at (166.0, 91.7)
- removed the R58 at (166.1, 104.9)
- added C25: 0.1u, Capacitor_SMD:C_0603_1608Metric_Pad1.08x0.95mm_HandSolder, F.Cu at (181.4, 64.8)
- added C26: 0.1u, Capacitor_SMD:C_0603_1608Metric_Pad1.08x0.95mm_HandSolder, F.Cu at (181.3, 118.4)
- added C27: 0.1u, Capacitor_SMD:C_0603_1608Metric_Pad1.08x0.95mm_HandSolder, F.Cu at (181.3, 91.4)
- added C52: 0.1u, Capacitor_SMD:C_0603_1608Metric_Pad1.08x0.95mm_HandSolder, B.Cu at (197.6, 114.4)
- added C53: 0.1u, Capacitor_SMD:C_0603_1608Metric_Pad1.08x0.95mm_HandSolder, B.Cu at (197.6, 89.8)
- added C54: 0.1u, Capacitor_SMD:C_0603_1608Metric_Pad1.08x0.95mm_HandSolder, B.Cu at (197.9, 64.4)
- added R44: 47, Resistor_SMD:R_0603_1608Metric_Pad0.98x0.95mm_HandSolder, F.Cu at (175.4, 108.0)
- added R46: 47, Resistor_SMD:R_0603_1608Metric_Pad0.98x0.95mm_HandSolder, F.Cu at (175.3, 81.3)
- added R51: 24k, Resistor_SMD:R_0603_1608Metric_Pad0.98x0.95mm_HandSolder, F.Cu at (199.0, 77.7)
- added R62: 47, Resistor_SMD:R_0603_1608Metric_Pad0.98x0.95mm_HandSolder, F.Cu at (175.2, 67.8)
- C46: renamed from C43; value 0.01u -> 0.1u; moved to F.Cu
- C47: renamed from C44; value 0.01u -> 0.1u; moved to F.Cu
- C48: renamed from C45; value 0.01u -> 0.1u; moved to F.Cu
- C49: renamed from C46; value 0.01u -> 0.1u; moved to F.Cu
- C50: renamed from C47; value 0.01u -> 0.1u; moved to F.Cu
- C51: renamed from C48; value 0.01u -> 0.1u; moved to F.Cu
- C56: renamed from C50; value 0.01u -> 0.1u; moved to F.Cu
- C57: renamed from C51; value 0.01u -> 0.1u; moved to F.Cu
- C58: renamed from C52; value 0.01u -> 0.1u; moved to F.Cu
- C59: renamed from C53; value 0.01u -> 0.1u; moved to F.Cu
- C60: renamed from C54; value 0.01u -> 0.1u; moved to F.Cu
- C61: renamed from C55; value 0.01u -> 0.1u; moved to F.Cu
- Q1, Q10, Q11, Q12, Q2, Q3, Q4, Q5, Q6, Q7, Q8, Q9: value MTB7D0N6RJ3 -> TPH4R008QM; footprint Package_TO_SOT_SMD:TO-252-2 -> MyLib:8-SOP Advance (5x5.75)
- R43: renamed from R46; moved to F.Cu
- R45: renamed from R48; moved to F.Cu
- R47: renamed from R50; moved to F.Cu
- R48: renamed from R51; moved to F.Cu
- R52, R53, R54: value surge_absorber -> 120; footprint Resistor_THT:R_Axial_DIN0207_L6.3mm_D2.5mm_P10.16mm_Horizontal -> Resistor_SMD:R_0603_1608Metric_Pad0.98x0.95mm_HandSolder; moved to B.Cu
- R57: renamed from R55; moved to F.Cu
- R58: renamed from R56; moved to F.Cu
- R59: renamed from R57; moved to F.Cu
- R60: moved to F.Cu
- R61: renamed from R59; moved to F.Cu
- moved R60 18.5 mm to (175.3, 94.2)
- moved C22 15.2 mm to (181.5, 104.9)
- moved C23 15.0 mm to (181.5, 78.2)
- moved C51 14.7 mm to (173.4, 52.6), turned to 0 degrees
- moved C59 14.7 mm to (173.5, 92.7), turned to 0 degrees
- moved C49 14.6 mm to (173.5, 79.8), turned to 0 degrees
- moved C61 14.6 mm to (173.4, 66.3), turned to 0 degrees
- moved C47 14.3 mm to (173.6, 106.4), turned to 0 degrees
- moved R48 14.1 mm to (175.2, 54.1)
- moved C57 14.0 mm to (173.4, 119.9), turned to 0 degrees
- moved C24 13.9 mm to (180.0, 52.3)
- moved R58 13.5 mm to (175.2, 121.4)
- moved R57 13.1 mm to (184.0, 119.9), turned to 180 degrees
- moved R61 12.9 mm to (184.0, 66.3), turned to 180 degrees
- moved R59 12.7 mm to (184.3, 93.0), turned to 180 degrees
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- renumbered C25 to C28, C26 to C29, C27 to C30, C28 to C31, C29 to C32, C30 to C33, C31 to C34, C32 to C35, C33 to C36, C34 to C37, C35 to C38, C36 to C39, C37 to C40, C38 to C41, C39 to C42, C40 to C43, C41 to C44, C42 to C45, C49 to C55, C56 to C62, C57 to C63, C58 to C64, C59 to C65, C60 to C66, C61 to C67, C62 to C68, C63 to C69, C64 to C70, C65 to C71, C66 to C72, C67 to C73, C68 to C74, C69 to C75, C70 to C76, C71 to C77, C72 to C78, C73 to C79, C74 to C80, C75 to C81, C76 to C82, C77 to C83, C78 to C84, D49 to D43, D50 to D44, D51 to D45, D52 to D46, D53 to D47, D54 to D48, D61 to D49, D62 to D50, D63 to D51, D64 to D52, D65 to D53, D66 to D54, D67 to D55, D68 to D56, D69 to D57, D70 to D58, D71 to D59, D72 to D60, D73 to D61, D74 to D62, D75 to D63, D76 to D64, D77 to D65, D78 to D66, D79 to D67, D80 to D68, D81 to D69, D82 to D70, D83 to D71, D84 to D72, D85 to D73, D86 to D74, D87 to D75, R43 to R49, R44 to R50, R61 to R55, R62 to R56
Connections:
- C20 pad 1: +5VD -> +3V3
- C59 pad 2: Net-(D58-K) (its old number) -> Net-(C59-Pad2)
- C61 pad 2: Net-(D60-K) (its old number) -> Net-(C61-Pad2)
- D49 pad 2: Net-(D61-A) -> Net-(D49-A)
- D50 pad 2: Net-(D62-A) -> Net-(D50-A)
- D51 pad 2: Net-(D63-A) -> Net-(D51-A)
- D52 pad 2: Net-(D64-A) -> Net-(D52-A)
- D53 pad 2: Net-(D65-A) -> Net-(D53-A)
- D54 pad 2: Net-(D66-A) -> Net-(D54-A)
- J7 pad : GND -> VCC
- J8 pad : GND -> VCC
- J9 pad : GND -> VCC
- Q1 pad 1: Net-(D37-A) -> Source_1A
- Q1 pad 2: VCC -> Source_1A
- Q10 pad 1: Net-(D65-A) -> GND
- Q10 pad 2: Source_2B -> GND
- Q11 pad 1: Net-(D63-A) -> Source_3B
- Q11 pad 2: VCC -> Source_3B
- Q12 pad 1: Net-(D66-A) -> GND
- Q12 pad 2: Source_3B -> GND
- Q2 pad 1: Net-(D38-A) -> GND
- Q2 pad 2: Source_1A -> GND
- Q3 pad 1: Net-(D39-A) -> Source_2A
- Q3 pad 2: VCC -> Source_2A
- Q4 pad 1: Net-(D40-A) -> GND
- Q4 pad 2: Source_2A -> GND
- Q5 pad 1: Net-(D41-A) -> Source_3A
- Q5 pad 2: VCC -> Source_3A
- Q6 pad 1: Net-(D42-A) -> GND
- Q6 pad 2: Source_3A -> GND
- Q7 pad 1: Net-(D61-A) -> Source_1B
- Q7 pad 2: VCC -> Source_1B
- Q8 pad 1: Net-(D64-A) -> GND
- Q8 pad 2: Source_1B -> GND
- Q9 pad 1: Net-(D62-A) -> Source_2B
- Q9 pad 2: VCC -> Source_2B
- R52 pad 1: Source_1A -> Source_1B
- R52 pad 2: Source_1B -> Net-(C52-Pad2)
- R53 pad 1: Source_2A -> Source_2B
- R53 pad 2: Source_2B -> Net-(C53-Pad2)
- R54 pad 1: Source_3A -> Source_3B
- R54 pad 2: Source_3B -> Net-(C54-Pad2)
- R60 pad 1: Source_3B -> Source_2B
- R60 pad 2: Net-(D60-K) (its old number) -> Net-(C59-Pad2)
- R63 pad 2: Net-(D61-A) -> Net-(D49-A)
- R64 pad 2: Net-(D64-A) -> Net-(D52-A)
- R65 pad 2: Net-(D62-A) -> Net-(D50-A)
- R66 pad 2: Net-(D65-A) -> Net-(D53-A)
- R67 pad 2: Net-(D63-A) -> Net-(D51-A)
- R68 pad 2: Net-(D66-A) -> Net-(D54-A)
- R69 pad 2: Net-(D61-A) -> Net-(D49-A)
- R70 pad 2: Net-(D62-A) -> Net-(D50-A)
- R71 pad 2: Net-(D63-A) -> Net-(D51-A)
- R72 pad 2: Net-(D64-A) -> Net-(D52-A)
- R73 pad 2: Net-(D65-A) -> Net-(D53-A)
- R74 pad 2: Net-(D66-A) -> Net-(D54-A)
- U6 pad 1: +5VD -> +3V3
Routing:
- net GND: track 876.0 -> 402.6 mm, vias 932 -> 1305
- net Net-(D50-A): track 0.00 -> 37.4 mm, vias 0 -> 2
- net Net-(D51-A): track 0.00 -> 37.1 mm, vias 0 -> 2
- net Net-(D49-A): track 0.00 -> 36.3 mm, vias 0 -> 2
- net +3V3: track 208.8 -> 235.0 mm, vias 3 -> 5
- net Net-(D62-A): track 23.6 -> 0.00 mm
- net VCC: track 208.1 -> 231.4 mm, vias 56 -> 277
- net Net-(D61-A): track 23.3 -> 0.00 mm
- net Net-(D63-A): track 23.2 -> 0.00 mm
- net Net-(D53-A): track 0.00 -> 21.9 mm, vias 0 -> 2
- net Net-(D54-A): track 0.00 -> 21.8 mm, vias 0 -> 2
- net Net-(D52-A): track 0.00 -> 21.6 mm, vias 0 -> 2
- net Source_2B: track 39.4 -> 54.4 mm, vias 230 -> 363
- net Source_1B: track 40.0 -> 54.7 mm, vias 235 -> 330
- net Net-(D64-A): track 14.7 -> 0.00 mm
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Other:
- board text added: "DCMotor Driver Rev3.1 @KayOChef_meme"
- board text removed: "DCMotor Driver Rev3.0 @KayOChef_meme"
