File: MD_Stable.kicad_pcb (KiCad board)
At the start: 2 copper layers, 100 x 100 mm, 304 parts, among them J1 XT30_Male, J10 Conn_01x08_Pin, J11 Conn_01x05_Socket, J2 XT60_Male, J3 RE1, J4 RE2, J5 RE3, J6 MO_XT60_Female1, J7 MO_XT60_Female2, J8 MO_XT60_Female3, J9 Conn_02x06_Odd_Even, Q1 AGM028N08A, Q10 AGM028N08A, Q11 AGM028N08A, Q12 AGM028N08A, Q2 AGM028N08A, Q3 AGM028N08A, Q4 AGM028N08A, Q5 AGM028N08A, Q6 AGM028N08A, Q7 AGM028N08A, Q8 AGM028N08A, Q9 AGM028N08A, SW1 SW_Push, SW2 SW_Push, SW3 SW_DIP_x03, SW4 PWM, SW5 PWM, SW6 PWM, SW7 DIR, SW8 DIR, SW9 DIR, U1 NJM7815SDL1, U10 74AHC1G08W5, U11 74AHC1G08W5, U12 74AHC1G08W5, U13 IR2184, U14 IR2184, U15 IR2184, U16 NE555D, U17 IR2184, U18 IR2184, U19 IR2184, U2 BA05CC0Tに似た何か, U20 74AHC1G08W5, U21 74AHC1G08W5, U22 74AHC1G08W5, U23 UTRS485G-S08-R, U24 UTRS485G-S08-R, U3 STM32G431K8Tx, U4 BA05CC0Tに似た何か, U5 BA033CC0FP, U6 π160M60, U7 74AHC1G04W5, U8 74AHC1G04W5, U9 74AHC1G04W5

Commit message: 時代はね、CANなんすよ
Parts:
- removed the C82 at (118.5, 80.3)
- removed the C84 at (118.7, 96.3)
- removed R78: 120, Resistor_SMD:R_0603_1608Metric_Pad0.98x0.95mm_HandSolder
- removed R79, R80, R81, R82: 2.2k, Resistor_SMD:R_0603_1608Metric_Pad0.98x0.95mm_HandSolder
- removed U24: UTRS485G-S08-R, Package_SO:SOP-8_3.76x4.96mm_P1.27mm
- added C1: 22p, Capacitor_SMD:C_0603_1608Metric_Pad1.08x0.95mm_HandSolder, B.Cu at (113.9, 88.6)
- added C3: 22p, Capacitor_SMD:C_0603_1608Metric_Pad1.08x0.95mm_HandSolder, B.Cu at (108.9, 88.6)
- added C83: 0.1u, Capacitor_SMD:C_0603_1608Metric_Pad1.08x0.95mm_HandSolder, F.Cu at (113.5, 86.7)
- added C85: 0.1u, Capacitor_SMD:C_0603_1608Metric_Pad1.08x0.95mm_HandSolder, F.Cu at (116.1, 86.7)
- added Y1: 8MHz, Crystal:Crystal_HC49-U_Vertical, F.Cu at (114.9, 92.2)
- J11: value Conn_01x05_Socket -> FDCAN_1; footprint Connector_JST:JST_XH_S5B-XH-A-1_1x05_P2.50mm_Horizontal -> Connector_JST:JST_XH_S2B-XH-A_1x02_P2.50mm_Horizontal
- U23: value UTRS485G-S08-R -> MCP2562-E-P
- moved R77 3.91 mm to (111.3, 83.7)
- moved J11 0.80 mm to (109.0, 82.5)
- moved U23 0.53 mm to (116.1, 83.9)
- renumbered C8 to C10, C9 to C11, C10 to C12, C11 to C13, C12 to C14, C13 to C15, C14 to C16, C15 to C17, C16 to C18, C17 to C19, C1 to C2, C18 to C20, C19 to C21, C20 to C22, C21 to C23, C22 to C24, C23 to C25, C24 to C26, C25 to C27, C26 to C28, C27 to C29, C28 to C30, C29 to C31, C30 to C32, C31 to C33, C32 to C34, C33 to C35, C34 to C36, C35 to C37, C36 to C38, C37 to C39, C2 to C4, C38 to C40, C39 to C41, C40 to C42, C41 to C43, C42 to C44, C43 to C45, C44 to C46, C45 to C47, C46 to C48, C47 to C49, C3 to C5, C48 to C50, C49 to C51, C50 to C52, C51 to C53, C52 to C54, C53 to C55, C54 to C56, C55 to C57, C56 to C58, C57 to C59, C4 to C6, C58 to C60, C59 to C61, C60 to C62, C61 to C63, C62 to C64, C63 to C65, C64 to C66, C65 to C67, C66 to C68, C67 to C69, C5 to C7, C68 to C70, C69 to C71, C70 to C72, C71 to C73, C72 to C74, C73 to C75, C74 to C76, C75 to C77, C76 to C78, C77 to C79, C6 to C8, C78 to C80, C79 to C81, C80 to C82, C81 to C84, C83 to C86, C7 to C9, D11 to D10, D9 to D11, D14 to D12, D12 to D13, D15 to D14, D13 to D15, D17 to D16, D18 to D17, D16 to D18, D4 to D3, D3 to D4, D10 to D9, R2 to R1, R12 to R11, R13 to R12, R11 to R13, R16 to R15, R17 to R16, R18 to R17, R19 to R18, R20 to R19, R1 to R2, R15 to R20, R22 to R21, R23 to R22, R24 to R23, R21 to R24, R4 to R3, R5 to R4, R6 to R5, R3 to R6, R9 to R7, R7 to R8, R8 to R9, SW3 to SW2, SW2 to SW3
Connections:
- J11 pad 1: GNDD -> Net-(J11-Pin_1)
- J9 pad 10: MCO_IN -> unconnected-(J9-Pin_10-Pad10)
- R77 pad 1: Net-(J11-Pin_2) -> Net-(J11-Pin_1)
- R77 pad 2: Net-(J11-Pin_3) -> Net-(J11-Pin_2)
- U23 pad 1: unconnected-(U23-RO-Pad1) -> FDCAN_TX
- U23 pad 2: RS485_DE -> GNDD
- U23 pad 3: RS485_DE -> +5VD
- U23 pad 4: RS485_TX -> FDCAN_RX
- U23 pad 5: GNDD -> +3V3
- U23 pad 7: Net-(J11-Pin_3) -> Net-(J11-Pin_1)
- U23 pad 8: +5VD -> GNDD
- U3 pad 2: MCO_IN -> Net-(U3-PF0)
- U3 pad 21: RE1_A -> FDCAN_RX
- U3 pad 22: RE1_B -> FDCAN_TX
- U3 pad 29: RS485_TX -> RE1_A
- U3 pad 3: RS485_DE -> Net-(U3-PF1)
- U3 pad 30: RS485_RX -> RE1_B
Routing:
- net MCO_IN: track 74.6 -> 0.00 mm, vias 1 -> 0
- net Net-(U3-PF1): track 0.00 -> 37.4 mm, vias 0 -> 1
- net Net-(U3-PF0): track 0.00 -> 35.7 mm, vias 0 -> 1
- net FDCAN_TX: track 0.00 -> 33.9 mm, vias 0 -> 1
- net RS485_DE: track 33.7 -> 0.00 mm, vias 1 -> 0
- net FDCAN_RX: track 0.00 -> 31.6 mm, vias 0 -> 1
- net RS485_TX: track 23.9 -> 0.00 mm, vias 1 -> 0
- net +3V3: track 234.9 -> 256.8 mm, vias 5 -> 6
- net RS485_RX: track 19.2 -> 0.00 mm, vias 1 -> 0
- net Net-(J11-Pin_3): track 16.3 -> 0.00 mm
- net Net-(J11-Pin_4): track 15.0 -> 0.00 mm, vias 1 -> 0
- net +5VD: track 210.2 -> 197.3 mm, vias 7 -> 5
- net Net-(J11-Pin_5): track 9.98 -> 0.00 mm, vias 1 -> 0
- net Net-(J11-Pin_2): track 9.68 -> 4.77 mm, vias 1 -> 0
- net Net-(J11-Pin_1): track 0.00 -> 4.89 mm
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Other:
- board text added: "<-CANH"
- board text added: "<-CANL"
- board text removed: "->RX:A"
- board text removed: "->RX:B"
- board text removed: "<-TX:A"
- board text removed: "<-TX:B"
