File: MD_Stable.kicad_sch (KiCad schematic)
At the start: 144 parts, among them J2 Conn_02x04_Counter_Clockwise, J6 Conn_01x03_Pin, J7 Conn_01x06_Socket, U11 TLP291, U12 TLP291, U8 NE555D

Commit message: 電装班がGitHubに上陸
Parts:
- added U1: STM32G431K8Tx, Package_QFP:LQFP-32_7x7mm_P0.8mm, symbol MCU_ST_STM32G4:STM32G431K8Tx
Connections:
- new net: U1.16 (VSS), U1.32 (VSS)
Changed lines of the file:
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@@
+	)
+	(symbol
+		(lib_id "MCU_ST_STM32G4:STM32G431K8Tx")
+		(at -20.32 227.33 0)
+		(unit 1)
+		(exclude_from_sim no)
+		(in_bom yes)
+		(on_board yes)
+		(dnp no)
+		(fields_autoplaced yes)
+		(property "Reference" "U1"
+			(at -15.6367 252.73 0)
+			(effects
+				(font
+					(size 1.27 1.27)
+				)
+				(justify left)
+			)
+		)
+		(property "Value" "STM32G431K8Tx"
+			(at -15.6367 255.27 0)
+			(effects
+				(font
+					(size 1.27 1.27)
+				)
+				(justify left)
+			)
+		)
+		(property "Footprint" "Package_QFP:LQFP-32_7x7mm_P0.8mm"
+			(at -30.48 250.19 0)
+			(effects
+				(font
+					(size 1.27 1.27)
+				)
+				(justify right)
+				(hide yes)
+			)
+		)
+		(property "Datasheet" "https://www.st.com/resource/en/datasheet/stm32g431k8.pdf"
+			(at -20.32 227.33 0)
+			(effects
+				(font
+					(size 1.27 1.27)
+				)
+				(hide yes)
+			)
+		)
+		(property "Description" "STMicroelectronics Arm Cortex-M4 MCU, 64KB flash, 32KB RAM, 170 MHz, 1.71-3.6V, 26 GPIO, LQFP32"
+			(at -20.32 227.33 0)
+			(effects
+				(font
+					(size 1.27 1.27)
+				)
+				(hide yes)
+			)
+		)
+		(pin "7"
+		)
+		(pin "10"
+		)
+		(pin "20"
+		)
+		(pin "1"
+		)
+		(pin "28"
+		)
+		(pin "3"
+		)
+		(pin "27"
+		)
+		(pin "30"
+		)
+		(pin "17"
+		)
+		(pin "5"
+		)
+		(pin "14"
+		)
+		(pin "11"
+		)
+		(pin "8"
+		)
+		(pin "31"
+		)
+		(pin "16"
+		)
+		(pin "12"
+		)
+		(pin "2"
+		)
+		(pin "26"
+		)
+		(pin "19"
+		)
+		(pin "15"
+		)
+		(pin "13"
+		)
+		(pin "29"
+		)
+		(pin "32"
+		)
+		(pin "6"
+		)
+		(pin "4"
+		)
+		(pin "9"
+		)
+		(pin "18"
+		)
+		(pin "21"
+		)
+		(pin "23"
+		)
+		(pin "22"
+		)
+		(pin "24"
+		)
+		(pin "25"
+		)
+		(instances
+			(project ""
+				(path "/3c9b7a20-e029-4fdf-87dd-ccce7ab9baef"
+					(reference "U1")
+					(unit 1)
+				)
+			)
+		)
 	)
 	(symbol

Commit message: 回路図おおむね完成
Parts:
- removed C?: 16v 100u, Capacitor_THT:CP_Radial_D5.0mm_P2.00mm, symbol Device:C_Polarized
- removed C? (x2): 0.1u, Capacitor_SMD:C_0603_1608Metric_Pad1.08x0.95mm_HandSolder, symbol Device:C
- removed D? (x6): 1N4148W, Diode_SMD:D_SOD-123, symbol Diode:1N4007
- removed D?: LED, LED_SMD:LED_0603_1608Metric_Pad1.05x0.95mm_HandSolder, symbol Device:LED
- removed J6: Conn_01x03_Pin, Connector_PinHeader_2.54mm:PinHeader_1x03_P2.54mm_Horizontal, symbol Connector:Conn_01x03_Pin
- removed J7: Conn_01x06_Socket, Connector_JST:JST_XH_S6B-XH-A_1x06_P2.50mm_Horizontal, symbol Connector:Conn_01x06_Socket
- removed J?: Conn_02x05_Odd_Even, Connector_PinSocket_2.54mm:PinSocket_2x05_P2.54mm_Horizontal, symbol Connector_Generic:Conn_02x05_Odd_Even
- removed R36, R? (x4): 10k, Resistor_SMD:R_0603_1608Metric_Pad0.98x0.95mm_HandSolder, symbol Device:R
- removed R37, R38, R40, R?: 1k, Resistor_SMD:R_0603_1608Metric_Pad0.98x0.95mm_HandSolder, symbol Device:R
- removed R39: 2k, Resistor_SMD:R_0603_1608Metric_Pad0.98x0.95mm_HandSolder, symbol Device:R
- removed SW?: SW_Push, Button_Switch_THT:SW_PUSH_6mm_H4.3mm, symbol Switch:SW_Push
- removed U11, U12: TLP291, Package_SO:SOIC-4_4.55x2.6mm_P1.27mm, symbol Isolator:TLP291
- removed U?: 74AHC1G08W5, Package_TO_SOT_SMD:SOT-23-5_HandSoldering, symbol 4xxx:4081
- removed U?: 74AHC1G04W5, Package_TO_SOT_SMD:SOT-23-5_HandSoldering, symbol 4xxx:4069
- removed U?: BA033CC0FP, Package_TO_SOT_SMD:TO-252-2, symbol Regulator_Linear:LF33_TO252
- removed U?: STM32F303K8Tx, Package_QFP:LQFP-32_7x7mm_P0.8mm, symbol MCU_ST_STM32F3:STM32F303K8Tx
- added C? (x16): 1u, Capacitor_SMD:C_0603_1608Metric_Pad1.08x0.95mm_HandSolder, symbol Device:C
- added C? (x6): 0.22u, Capacitor_SMD:C_0603_1608Metric_Pad1.08x0.95mm_HandSolder, symbol Device:C
- added C? (x17): 0.1u, Capacitor_SMD:C_0603_1608Metric_Pad1.08x0.95mm_HandSolder, symbol Device:C
- added C? (x8): 0.01u, Capacitor_SMD:C_0603_1608Metric_Pad1.08x0.95mm_HandSolder, symbol Device:C
- added C?: 16V 100u, Capacitor_THT:CP_Radial_D5.0mm_P2.00mm, symbol Device:C_Polarized
- added C?: 50v 100u, Capacitor_THT:CP_Radial_D8.0mm_P3.50mm, symbol Device:C_Polarized
- added C?: 16v 100u, Capacitor_THT:CP_Radial_D5.0mm_P2.00mm, symbol Device:C_Polarized
- added D? (x44): 1N4148W, Diode_SMD:D_SOD-123, symbol Diode:1N4007
- added D? (x4): UDZVTE-1715B, Diode_SMD:D_SOD-323_HandSoldering, symbol Device:D_Zener
- added D? (x3): LED, LED_SMD:LED_0603_1608Metric_Pad1.05x0.95mm_HandSolder, symbol Device:LED
- added D? (x2): LED_A, LED_SMD:LED_0603_1608Metric_Pad1.05x0.95mm_HandSolder, symbol Device:LED
- added D? (x8): GS1010FL, Diode_SMD:D_SOD-123F, symbol Diode:1N4007
- added D? (x2): LED_B, LED_SMD:LED_0603_1608Metric_Pad1.05x0.95mm_HandSolder, symbol Device:LED
- added J?: XT30_Male, Connector_AMASS:AMASS_XT60PW-M_1x02_P7.20mm_Horizontal, symbol Connector:Conn_01x02_Pin
- added J?: Conn_01x04_Socket, symbol Connector:Conn_01x04_Socket
- added J? (x2): MO_XT60_Female, Connector_AMASS:AMASS_XT60PW-F_1x02_P7.20mm_Horizontal, symbol Connector:Conn_01x02_Socket
- added J?: Conn_01x08_Pin, symbol Connector:Conn_01x08_Pin
- added J? (x2): RE, MyLib:PocketHeader_1x05_Horizontal, symbol Connector:Conn_01x05_Socket
- added J?: Conn_02x06_Odd_Even, symbol Connector_Generic:Conn_02x06_Odd_Even
- added Q? (x8): MTB7D0N6RJ3, Package_TO_SOT_SMD:TO-252-2, symbol Simulation_SPICE:NMOS
- added R? (x16): 10k, Resistor_SMD:R_0603_1608Metric_Pad0.98x0.95mm_HandSolder, symbol Device:R
- added R? (x16): 47, Resistor_SMD:R_0603_1608Metric_Pad0.98x0.95mm_HandSolder, symbol Device:R
- added R? (x8): 47k, Resistor_SMD:R_0603_1608Metric_Pad0.98x0.95mm_HandSolder, symbol Device:R
- added R? (x2): surge_absorber, Resistor_THT:R_Axial_DIN0207_L6.3mm_D2.5mm_P10.16mm_Horizontal, symbol Device:R
- added R? (x3): 24k, Resistor_SMD:R_0603_1608Metric_Pad0.98x0.95mm_HandSolder, symbol Device:R
- added R? (x2): 1k, Resistor_SMD:R_0603_1608Metric_Pad0.98x0.95mm_HandSolder, symbol Device:R
- added SW? (x2): PWM, Button_Switch_THT:SW_PUSH_6mm_H4.3mm, symbol Switch:SW_Push
- added SW? (x2): DIR, Button_Switch_THT:SW_PUSH_6mm_H4.3mm, symbol Switch:SW_Push
- added SW?: SW_Push, Button_Switch_THT:SW_PUSH_6mm_H4.3mm, symbol Switch:SW_Push
- added U? (x5): 74AHC1G08W5, Package_TO_SOT_SMD:SOT-23-5_HandSoldering, symbol 4xxx:4081
- added U?: BA033CC0FP, Package_TO_SOT_SMD:TO-252-2, symbol Regulator_Linear:LF33_TO252
- added U? (x3): 74AHC1G04W5, Package_TO_SOT_SMD:SOT-23-5_HandSoldering, symbol 4xxx:4069
- added U? (x4): IRS2302S, Package_SO:SOIC-8_3.9x4.9mm_P1.27mm, symbol Driver_FET:IRS2302S
- added U?: π160M60, Package_SO:SOIC-16W_7.5x10.3mm_P1.27mm, symbol MyLib:π160M60
- added U?: BA05CC0Tに似た何か, Package_TO_SOT_SMD:TO-252-2, symbol Regulator_Linear:LF33_TO252
- C? (x4): value 0.1u -> 0.01u
- R?: value 1k -> 10k
- U?: value NJM7812SDL1 -> NJM7808SDL1
- renumbered D27 to D?, D20 to D?, J2 to J?, R26 to R?, U1 to U?, U8 to U?
Connections:
- net GND1 is gone; now on net GNDD: C?.2, C?.2, R?.1, R?.1, U?.2 (~{RE}), U?.3 (DE), U?.5 (GND), U?.5 (GND)
- net +12V: now also C?.1, C?.1, C?.1, D?.1 (K), J?.2 (Pin_2), R?.2, U?.1 (VI); no longer C?.1, C?.1, C?.1, C?.1, C?.1, C?.1, D?.1 (K), D?.2 (A), D?.2 (A), D?.2 (A), R?.1, R?.1, R?.2, U?.1 (VCC), U?.1 (VCC), U?.3 (VO), U?.8 (VCC)
- net +3V3: now also U?.1 (VDD), U?.15 (VDDA), U?.17 (VDD), C?.1, C?.1, C?.1, D?.1 (K), D?.2 (A), J?.1 (Pin_1), R?.2, R?.2, U?.3 (VO); no longer R?.1, R?.1, SW?.1, SW?.1, U?.5 (VCC)
- net +5V: now also R?.1, R?.1, U?.5 (VCC), C?.1, R?.1, R?.1, R?.1, R?.1, U?.16 (VDD2), U?.5 (VCC), U?.5 (VCC), U?.5 (VCC), U?.5 (VCC), U?.5 (VCC), U?.5 (VCC), U?.5 (VCC), U?.5 (VCC); no longer C?.1, J?.4 (Pin_4), R?.2, R?.2
- net +5VA: no longer C?.1, R?.2, R?.2, U?.2 (~{RE}), U?.3 (DE), U?.8 (VCC), U?.8 (VCC)
- net 555_Out_A: now also C?.2, C?.2, C?.2, C?.2, C?.2, C?.2, C?.2, C?.2
- net DIP_1: now also U?.11 (PA6)
- net DIP_2: now also U?.10 (PA5)
- net DIP_3: now also U?.9 (PA4)
- net DIP_4: now also U?.3 (PF1)
- net DIR1: now also D?.1 (K), J?.2 (Pin_2), R?.2, U?.7 (Vif); no longer U?.1 (A)
- net GND: now also C?.1, C?.1, C?.1, C?.1, C?.1, C?.1, C?.1, C?.1, C?.1, C?.1, C?.1, C?.1, C?.1, C?.1, C?.2, C?.2, C?.2, C?.2, C?.2, C?.2, C?.2, C?.2, Q?.3 (S), Q?.3 (S), Q?.3 (S), Q?.3 (S), R?.1, R?.1, R?.1, R?.1, U?.3 (GND), U?.3 (GND), U?.3 (GND), U?.3 (GND), U?.3 (GND), U?.3 (GND), U?.3 (GND), U?.3 (GND), U?.4 (COM), U?.4 (COM), U?.4 (COM), U?.4 (COM), U?.9 (GND2); no longer C?.2, C?.2, C?.2, C?.2, D?.1 (K), J?.1 (Pin_1), R?.1, R?.1, R?.1, R?.1, SW?.2
- net LED_1: now also U?.31 (PB8), R?.2
- net MCO_IN: now also U?.2 (PF0), J?.10 (Pin_10)
- net PWM1: now also D?.1 (K), J?.3 (Pin_3), R?.2, U?.6 (Vie); no longer U?.2 (B)
- net RE1_A: now also U?.5 (PA0)
- net RE1_B: now also U?.6 (PA1)
- net RESET: now also U?.4 (PG10), J?.9 (Pin_9), R?.1, SW?.1
- net RS485_RX: now also U?.1 (RO), U?.30 (PB7)
- net RS485_TX: now also U?.29 (PB6), U?.4 (DI)
- net SWCLK: now also U?.24 (PA14), J?.3 (Pin_3)
- net SWDIO: now also U?.23 (PA13), J?.7 (Pin_7)
- net UART_RX: now also U?.8 (PA3), J?.6 (Pin_6)
- net UART_TX: now also U?.7 (PA2), J?.4 (Pin_4)
- net User_Button: now also U?.12 (PA7)
- net VCC: now also C?.1, C?.1, C?.1, C?.2, C?.2, C?.2, C?.2, D?.2 (A), D?.2 (A), D?.2 (A), D?.2 (A), D?.2 (A), D?.2 (A), Q?.2 (D), Q?.2 (D), Q?.2 (D), Q?.2 (D); no longer C?.1, D?.1 (K), U?.1 (VI)
- net Source_1A: now reaches D?.1 (K), D?.2 (A), D?.2 (A), J?.2 (Pin_2), Q?.2 (D), Q?.3 (S), R?.1, R?.1, R?.1, R?.2, R?.2, U?.6 (VS)
- net Source_1A: now also D?.2 (A), C?.1
- net Source_1B: now reaches D?.1 (K), D?.1 (K), D?.2 (A), D?.2 (A), D?.2 (A), J?.1 (Pin_1), Q?.2 (D), Q?.3 (S), R?.1, R?.1, R?.2, R?.2, U?.6 (VS)
- net Source_1B: now also D?.2 (A), C?.1
- net at U?.2 (IN): now also U?.4 (Y)
- net at U?.13 (PB0): now also D?.2 (A)
- net GNDD: now reaches U?.14 (VSSA)
- net GNDD: now also C?.2, C?.2, D?.1 (K), J?.1 (Pin_1), R?.1, R?.1, R?.1, R?.1, SW?.2, U?.16 (VSS), U?.32 (VSS), C?.2, C?.2, C?.2, C?.2, C?.2, C?.2, C?.2, C?.2, C?.2, C?.2, C?.2, C?.2, D?.1 (K), D?.1 (K), D?.1 (K), D?.2 (A), D?.2 (A), J?.1 (Pin_1), J?.1 (Pin_1), J?.1 (Pin_1), J?.12 (Pin_12), J?.5 (Pin_5), J?.8 (Pin_8), R?.1, R?.1, R?.1, R?.1, R?.1, R?.1, R?.1, SW?.2, U?.2 (GND), U?.2 (GND), U?.8 (GND1)
- net at U?.18 (PA8): now also D?.2 (A)
- net at U?.19 (PA9): now also D?.2 (A)
- net at U?.20 (PA10): now also D?.2 (A)
- net RE3_A: now reaches U?.21 (PA11)
- net RE3_A: now also J?.3 (Pin_3), R?.1
- net RE3_B: now reaches U?.22 (PA12)
- net RE3_B: now also J?.5 (Pin_5), R?.1
- net at U?.25 (PA15): now also D?.2 (A)
- net at U?.26 (PB3): now also D?.2 (A)
- net RE2_A: now reaches U?.27 (PB4)
- net RE2_A: now also J?.3 (Pin_3), R?.1
- net RE2_B: now reaches U?.28 (PB5)
- net RE2_B: now also J?.5 (Pin_5), R?.1
- net at D?.1 (K), U?.8 (VB): now also C?.2, C?.2, D?.1 (K); no longer C?.1 (x2)
- net at R?.1, R?.2, U?.7 (B): now also J?.2 (Pin_2)
- net at R?.1, R?.2, U?.6 (A): now also J?.3 (Pin_3)
- net at R?.1, R?.2, U?.7 (B): now also J?.4 (Pin_4)
- net at R?.1, R?.2, U?.6 (A): now also J?.1 (Pin_1)
- new net: C?.2, C?.2, D?.1 (K), D?.1 (K), U?.8 (VB) (x4)
- new net: C?.1, D?.1 (K), D?.2 (A) (x8)
- new net: C?.2, D?.1 (K), D?.2 (A) (x4)
- new net: R?.2, U?.3 (~{SD}) (x4)
- new net: D?.1 (K), D?.2 (A), Q?.1 (G), R?.2, R?.2 (x4)
- new net: D?.1 (K), R?.1, U?.7 (HO) (x4)
- new net: U?.2 (IN), U?.4 (Y) (x4)
- new net: D?.1 (K), R?.1, U?.5 (LO) (x4)
- new net: D?.2 (A), Q?.1 (G), R?.2, R?.2 (x4)
- new net: D?.2 (A), D?.2 (A), SW?.2 (x2)
- new net: C?.1, D?.2 (A), R?.1 (x4)
- new net: D?.2 (A), R?.1 (x3)
- new net: C?.1, C?.1, D?.1 (K), D?.2 (A), U?.1 (VI), U?.3 (VO)
- new net: C?.2, D?.1 (K), R?.2 (x4)
- new net: U?.1 (A), U?.4 (Y) (x3)
- new net: D?.1 (K), D?.2 (A), R?.1 (x2)
- new net +5VD: C?.1, C?.1, C?.1, C?.1, C?.1, C?.1, D?.1 (K), J?.1 (Pin_1), J?.4 (Pin_4), J?.4 (Pin_4), J?.4 (Pin_4), J?.8 (Pin_8), R?.2, R?.2, R?.2, R?.2, R?.2, R?.2, R?.2, R?.2, R?.2, SW?.1, SW?.1, SW?.1, SW?.1, SW?.1, SW?.1, U?.1 (VDD1), U?.2 (~{RE}), U?.3 (DE), U?.8 (VCC), U?.8 (VCC)
- new net +8V: C?.1, C?.1, C?.1, C?.1, C?.1, C?.1, C?.1, C?.1, C?.1, C?.1, C?.1, D?.1 (K), D?.1 (K), D?.2 (A), R?.1, R?.1, R?.2, U?.1 (VCC), U?.1 (VCC), U?.1 (VCC), U?.1 (VCC), U?.1 (VCC), U?.1 (VCC), U?.1 (VI), U?.3 (VO), U?.8 (VCC)
- new net DIR2: D?.1 (K), D?.1 (K), J?.4 (Pin_4), R?.2, U?.5 (Vid)
- new net DIR3: D?.1 (K), D?.1 (K), J?.6 (Pin_6), R?.2, U?.3 (Vib)
- new net PWM2: D?.1 (K), D?.1 (K), J?.5 (Pin_5), R?.2, SW?.2, U?.4 (Vic)
- new net PWM3: D?.1 (K), D?.1 (K), J?.7 (Pin_7), R?.2, SW?.2, U?.2 (Via)
- new net Source_2A: C?.1, D?.1 (K), D?.2 (A), D?.2 (A), D?.2 (A), J?.2 (Pin_2), Q?.2 (D), Q?.3 (S), R?.1, R?.1, R?.1, R?.2, R?.2, U?.6 (VS)
- new net Source_2B: C?.1, D?.1 (K), D?.1 (K), D?.2 (A), D?.2 (A), D?.2 (A), D?.2 (A), J?.1 (Pin_1), Q?.2 (D), Q?.3 (S), R?.1, R?.1, R?.2, R?.2, U?.6 (VS)
- new net Source_3A: C?.1, D?.1 (K), D?.2 (A), D?.2 (A), D?.2 (A), J?.2 (Pin_2), Q?.2 (D), Q?.3 (S), R?.1, R?.1, R?.1, R?.2, R?.2, U?.6 (VS)
- new net Source_3B: C?.1, D?.1 (K), D?.1 (K), D?.2 (A), D?.2 (A), D?.2 (A), D?.2 (A), J?.1 (Pin_1), Q?.2 (D), Q?.3 (S), R?.1, R?.1, R?.2, R?.2, U?.6 (VS)
- new net out_DIR1: U?.1 (A), U?.10 (Vof), U?.2 (A)
- new net out_DIR2: U?.1 (A), U?.12 (Vod), U?.2 (A)
- new net out_DIR3: U?.1 (A), U?.14 (Vob), U?.2 (A)
- new net out_PWM1: U?.11 (Voe), U?.2 (B), U?.2 (B)
- new net out_PWM2: U?.13 (Voc), U?.2 (B), U?.2 (B)
- new net out_PWM3: U?.15 (Voa), U?.2 (B), U?.2 (B)
- no-connect marks 14 -> 11
Other:
- note added: "G431K8"
- note added: "制御部VCC"
- note added: "制御部降圧"
- note added: "駆動部VCC"
- note added: "駆動部降圧"
- note removed: "F303K8"
- note removed: "VCC"
- note removed: "降圧"
- moved on the sheet: C?, D?, J?, Q?, R?, SW?, U?, U?A

Commit message: 配線し始めた
Parts:
- removed C?: 0.1u, Capacitor_SMD:C_0603_1608Metric_Pad1.08x0.95mm_HandSolder, symbol Device:C
- removed D? (x6): UDZVTE-1715B, Diode_SMD:D_SOD-323_HandSoldering, symbol Device:D_Zener
- removed J?: Conn_01x04_Socket, symbol Connector:Conn_01x04_Socket
- added J12: Conn_01x05_Socket, Connector_JST:JST_XH_S5B-XH-A-1_1x05_P2.50mm_Horizontal, symbol Connector:Conn_01x05_Socket
- J1: renamed from J?; footprint Package_DIP:DIP-8_W7.62mm -> Button_Switch_THT:SW_DIP_SPSTx04_Slide_6.7x11.72mm_W7.62mm_P2.54mm_LowProfile
- J10: renamed from J?; footprint (none) -> Connector_PinSocket_2.54mm:PinSocket_2x06_P2.54mm_Horizontal
- J11: renamed from J?; footprint (none) -> Connector_PinHeader_2.54mm:PinHeader_1x08_P2.54mm_Horizontal
- J2: renamed from J?; footprint Connector_AMASS:AMASS_XT60PW-M_1x02_P7.20mm_Horizontal -> Connector_AMASS:AMASS_XT30PW-M_1x02_P2.50mm_Horizontal
- J4: renamed from J?; value RE -> RE1
- J5: renamed from J?; value RE -> RE2
- J6: renamed from J?; value RE -> RE3
- J7: renamed from J?; value MO_XT60_Female -> MO_XT60_Female1
- J8: renamed from J?; value MO_XT60_Female -> MO_XT60_Female2
- J9: renamed from J?; value MO_XT60_Female -> MO_XT60_Female3
- SW1, SW2, SW3, SW4, SW5, SW6, SW7, SW8: renamed from SW?; footprint Button_Switch_THT:SW_PUSH_6mm_H4.3mm -> Button_Switch_THT:SW_PUSH_1P1T_6x3.5mm_H4.3_APEM_MJTP1243
- U23, U24: renamed from U?; footprint Package_SO:SOP-8_3.9x4.9mm_P1.27mm -> Package_SO:SOP-8_3.76x4.96mm_P1.27mm
- gave numbers to parts that had none: 283
Connections:
- net +5VA is gone; now on net +5VD: C77.1
- net +5VD: now also C5.1, C6.1, D10.1 (K), D4.2 (A), U2.3 (VO), U5.1 (VI)
- net DIR2: now also D3.1 (K), R3.2; no longer D12.1 (K), R12.2
- net DIR3: now also D12.1 (K), R12.2; no longer D3.1 (K), R3.2
- net GNDD: now also J12.5 (Pin_5)
- net PWM1: now also D9.1 (K), R16.2; no longer D16.1 (K), R26.2
- net PWM3: now also D16.1 (K), R26.2; no longer D9.1 (K), R16.2
- net RE1_A: now also U3.21 (PA11); no longer U3.5 (PA0)
- net RE1_B: now also U3.22 (PA12); no longer U3.6 (PA1)
- net RE2_A: now also U3.5 (PA0); no longer U3.27 (PB4)
- net RE2_B: now also U3.6 (PA1); no longer U3.28 (PB5)
- net RE3_A: now also U3.27 (PB4); no longer U3.21 (PA11)
- net RE3_B: now also U3.28 (PB5); no longer U3.22 (PA12)
- net at R78.1, R81.2, U23.6 (A): now also J12.1 (Pin_1)
- net at R78.2, R80.1, U23.7 (B): now also J12.2 (Pin_2)
- net at R79.1, R83.2, U24.6 (A): now also J12.3 (Pin_3)
- net at R79.2, R82.1, U24.7 (B): now also J12.4 (Pin_4)
Other:
- note added: "手動回転"
- note added: "絶縁"
- moved on the sheet: C12, C17, C9, D19, D8, D82, D83, D84, D85, D86, D87, SW3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

Commit message: 配線終わり見えてきた
Parts:
- added F1: Polyfuse, MyLib:PolyFuse_MF-NSMF-series, symbol Device:Polyfuse
Connections:
- net +12V: now also F1.1; no longer C2.1, D4.1 (K), U2.1 (VI)
- net GNDD: now also J12.1 (Pin_1); no longer J12.5 (Pin_5)
- net at R78.2, R80.1, U23.7 (B): now also J12.3 (Pin_3); no longer J12.2 (Pin_2)
- net at R79.1, R83.2, U24.6 (A): now also J12.4 (Pin_4); no longer J12.3 (Pin_3)
- net at R79.2, R82.1, U24.7 (B): now also J12.5 (Pin_5); no longer J12.4 (Pin_4)
- net at R78.1, R81.2, U23.6 (A): now also J12.2 (Pin_2); no longer J12.1 (Pin_1)
- new net: C2.1, D4.1 (K), F1.2, U2.1 (VI)
Other:
- moved on the sheet: J12
Changed lines of the file:
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@@
 	(wire
 		(pts
-			(xy 36.83 304.8) (xy 36.83 306.07)
+			(xy 25.4 304.8) (xy 25.4 306.07)
 		)
 		(stroke
@@
 	(wire
 		(pts
-			(xy 786.13 119.38) (xy 787.4 119.38)
+			(xy 786.13 106.68) (xy 787.4 106.68)
 		)
 		(stroke
@@
 	(wire
 		(pts
+			(xy 36.83 306.07) (xy 41.91 306.07)
+		)
+		(stroke
+			(width 0)
+			(type default)
+		)
+	)
+	(wire
+		(pts
 			(xy 97.79 149.86) (xy 108.585 149.86)
 		)
@@
 	(wire
 		(pts
-			(xy 36.83 306.07) (xy 41.91 306.07)
+			(xy 25.4 306.07) (xy 29.21 306.07)
 		)
 		(stroke
@@
 	(wire
 		(pts
-			(xy 786.13 124.46) (xy 786.13 119.38)
+			(xy 786.13 124.46) (xy 786.13 106.68)
 		)
 		(stroke
@@
 	)
 	(symbol
+		(lib_id "Device:Polyfuse")
+		(at 33.02 306.07 90)
+		(unit 1)
+		(exclude_from_sim no)
+		(in_bom yes)
+		(on_board yes)
+		(dnp no)
+		(fields_autoplaced yes)
+		(property "Reference" "F1"
+			(at 33.02 299.72 90)
+			(effects
+				(font
+					(size 1.27 1.27)
+				)
+			)
+		)
+		(property "Value" "Polyfuse"
+			(at 33.02 302.26 90)
+			(effects
+				(font
+					(size 1.27 1.27)
+				)
+			)
+		)
+		(property "Footprint" "MyLib:PolyFuse_MF-NSMF-series"
+			(at 38.1 304.8 0)
+			(effects
+				(font
+					(size 1.27 1.27)
+				)
+				(justify left)
+				(hide yes)
+			)
+		)
+		(property "Datasheet" "~"
+			(at 33.02 306.07 0)
+			(effects
+				(font
+					(size 1.27 1.27)
+				)
+				(hide yes)
+			)
+		)
+		(property "Description" "Resettable fuse, polymeric positive temperature coefficient"
+			(at 33.02 306.07 0)
+			(effects
+				(font
+					(size 1.27 1.27)
+				)
+				(hide yes)
+			)
+		)
+		(pin "1"
+		)
+		(pin "2"
+		)
+		(instances
+			(project ""
+				(path "/3c9b7a20-e029-4fdf-87dd-ccce7ab9baef"
+					(reference "F1")
+					(unit 1)
+				)
+			)
+		)
+	)
+	(symbol
 		(lib_id "Diode:1N4007")
 		(at 83.82 312.42 270)
@@
 	(symbol
 		(lib_id "Connector:Conn_01x05_Socket")
-		(at 792.48 114.3 0)
+		(at 792.48 111.76 0)
 		(unit 1)
 		(exclude_from_sim no)
@@
 		(fields_autoplaced yes)
 		(property "Reference" "J12"
-			(at 793.75 113.0299 0)
+			(at 793.75 110.4899 0)
 			(effects
 				(font
@@
 		)
 		(property "Value" "Conn_01x05_Socket"
-			(at 793.75 115.5699 0)
+			(at 793.75 113.0299 0)
 			(effects
 				(font
@@
 		)
 		(property "Footprint" "Connector_JST:JST_XH_S5B-XH-A-1_1x05_P2.50mm_Horizontal"
-			(at 792.48 114.3 0)
+			(at 792.48 111.76 0)
 			(effects
 				(font
@@
 		)
 		(property "Datasheet" "~"
-			(at 792.48 114.3 0)
+			(at 792.48 111.76 0)
 			(effects
 				(font
@@
 		)
 		(property "Description" "Generic connector, single row, 01x05, script generated"
-			(at 792.48 114.3 0)
+			(at 792.48 111.76 0)
 			(effects
 				(font
@@
 	(symbol
 		(lib_id "power:+12V")
-		(at 36.83 304.8 0)
+		(at 25.4 304.8 0)
 		(unit 1)
 		(exclude_from_sim no)
@@
 		(fields_autoplaced yes)
 		(property "Reference" "#PWR03"
-			(at 36.83 308.61 0)
+			(at 25.4 308.61 0)
 			(effects
 				(font
@@
 		)
 		(property "Value" "+12V"
-			(at 36.83 299.72 0)
+			(at 25.4 299.72 0)
 			(effects
 				(font
@@
 		)
 		(property "Footprint" ""
-			(at 36.83 304.8 0)
+			(at 25.4 304.8 0)
 			(effects
 				(font
@@
 		)
 		(property "Datasheet" ""
-			(at 36.83 304.8 0)
+			(at 25.4 304.8 0)
 			(effects
 				(font
@@
 		)
 		(property "Description" "Power symbol creates a global label with name \"+12V\""
-			(at 36.83 304.8 0)
+			(at 25.4 304.8 0)
 			(effects
 				(font

Commit message: rev3.1
Parts:
- removed D43, D44, D45, D46, D47, D48, D55, D56, D57, D58, D59, D60: GS1010FL, Diode_SMD:D_SOD-123F, symbol Diode:1N4007
- removed Q1, Q10, Q11, Q12, Q2, Q3, Q4, Q5, Q6, Q7, Q8, Q9: MTB7D0N6RJ3, Package_TO_SOT_SMD:TO-252-2, symbol Simulation_SPICE:NMOS
- added C25, C26, C27, C52, C53, C54: 0.1u, Capacitor_SMD:C_0603_1608Metric_Pad1.08x0.95mm_HandSolder, symbol Device:C
- added Q1, Q10, Q11, Q12, Q2, Q3, Q4, Q5, Q6, Q7, Q8, Q9: TPH4R008QM, MyLib:8-SOP Advance (5x5.75), symbol Transistor_FET:IRF7606PBF
- C46: renamed from C43; value 0.01u -> 0.1u
- C47: renamed from C44; value 0.01u -> 0.1u
- C48: renamed from C45; value 0.01u -> 0.1u
- C49: renamed from C46; value 0.01u -> 0.1u
- C50: renamed from C47; value 0.01u -> 0.1u
- C51: renamed from C48; value 0.01u -> 0.1u
- C56: renamed from C50; value 0.01u -> 0.1u
- C57: renamed from C51; value 0.01u -> 0.1u
- C58: renamed from C52; value 0.01u -> 0.1u
- C59: renamed from C53; value 0.01u -> 0.1u
- C60: renamed from C54; value 0.01u -> 0.1u
- C61: renamed from C55; value 0.01u -> 0.1u
- R52, R53, R54: value surge_absorber -> 120; footprint Resistor_THT:R_Axial_DIN0207_L6.3mm_D2.5mm_P10.16mm_Horizontal -> Resistor_SMD:R_0603_1608Metric_Pad0.98x0.95mm_HandSolder
- renumbered C25 to C28, C26 to C29, C27 to C30, C28 to C31, C29 to C32, C30 to C33, C31 to C34, C32 to C35, C33 to C36, C34 to C37, C35 to C38, C36 to C39, C37 to C40, C38 to C41, C39 to C42, C40 to C43, C41 to C44, C42 to C45, C49 to C55, C56 to C62, C57 to C63, C58 to C64, C59 to C65, C60 to C66, C61 to C67, C62 to C68, C63 to C69, C64 to C70, C65 to C71, C66 to C72, C67 to C73, C68 to C74, C69 to C75, C70 to C76, C71 to C77, C72 to C78, C73 to C79, C74 to C80, C75 to C81, C76 to C82, C77 to C83, C78 to C84, D49 to D43, D50 to D44, D51 to D45, D52 to D46, D53 to D47, D54 to D48, D61 to D49, D62 to D50, D63 to D51, D64 to D52, D65 to D53, D66 to D54, D67 to D55, D68 to D56, D69 to D57, D70 to D58, D71 to D59, D72 to D60, D73 to D61, D74 to D62, D75 to D63, D76 to D64, D77 to D65, D78 to D66, D79 to D67, D80 to D68, D81 to D69, D82 to D70, D83 to D71, D84 to D72, D85 to D73, D86 to D74, D87 to D75, R46 to R43, R47 to R44, R48 to R45, R49 to R46, R50 to R47, R51 to R48, R43 to R49, R44 to R50, R45 to R51, R61 to R55, R62 to R56, R55 to R57, R56 to R58, R57 to R59, R58 to R60, R59 to R61, R60 to R62
Connections:
- net +3V3: now also C20.1, U6.1 (VDD1)
- net +5VD: no longer C20.1, U6.1 (VDD1)
- net GND: now also C25.2, C26.2, C27.2, Q10.1 (S), Q10.2 (S), Q10.3 (S), Q12.1 (S), Q12.2 (S), Q12.3 (S), Q2.1 (S), Q2.2 (S), Q2.3 (S), Q4.1 (S), Q4.2 (S), Q4.3 (S), Q6.1 (S), Q6.2 (S), Q6.3 (S), Q8.1 (S), Q8.2 (S), Q8.3 (S)
- net Source_1A: now also C52.1, Q1.1 (S), Q1.2 (S), Q1.3 (S), Q2.5 (D), Q2.6 (D), Q2.7 (D), Q2.8 (D); no longer R52.1
- net Source_1B: now also R52.1, Q7.1 (S), Q7.2 (S), Q7.3 (S), Q8.5 (D), Q8.6 (D), Q8.7 (D), Q8.8 (D); no longer R52.2
- net Source_2A: now also C53.1, Q3.1 (S), Q3.2 (S), Q3.3 (S), Q4.5 (D), Q4.6 (D), Q4.7 (D), Q4.8 (D); no longer R53.1
- net Source_2B: now also R53.1, Q10.5 (D), Q10.6 (D), Q10.7 (D), Q10.8 (D), Q9.1 (S), Q9.2 (S), Q9.3 (S); no longer R53.2
- net Source_3A: now also C54.1, Q5.1 (S), Q5.2 (S), Q5.3 (S), Q6.5 (D), Q6.6 (D), Q6.7 (D), Q6.8 (D); no longer R54.1
- net Source_3B: now also R54.1, Q11.1 (S), Q11.2 (S), Q11.3 (S), Q12.5 (D), Q12.6 (D), Q12.7 (D), Q12.8 (D); no longer R54.2
- net VCC: now also C25.1, C26.1, C27.1, Q1.5 (D), Q1.6 (D), Q1.7 (D), Q1.8 (D), Q11.5 (D), Q11.6 (D), Q11.7 (D), Q11.8 (D), Q3.5 (D), Q3.6 (D), Q3.7 (D), Q3.8 (D), Q5.5 (D), Q5.6 (D), Q5.7 (D), Q5.8 (D), Q7.5 (D), Q7.6 (D), Q7.7 (D), Q7.8 (D), Q9.5 (D), Q9.6 (D), Q9.7 (D), Q9.8 (D)
- net at D39.2 (A), R32.2, R38.2: now also Q3.4 (G)
- net at D53.2 (A), R66.2, R73.2: now also Q10.4 (G)
- net at D40.2 (A), R33.2, R39.2: now also Q4.4 (G)
- net at D49.2 (A), R63.2, R69.2: now also Q7.4 (G)
- net at D42.2 (A), R35.2, R41.2: now also Q6.4 (G)
- net at D51.2 (A), R67.2, R71.2: now also Q11.4 (G)
- net at D38.2 (A), R31.2, R37.2: now also Q2.4 (G)
- net at D37.2 (A), R30.2, R36.2: now also Q1.4 (G)
- net at D50.2 (A), R65.2, R70.2: now also Q9.4 (G)
- net at D52.2 (A), R64.2, R72.2: now also Q8.4 (G)
- net at D54.2 (A), R68.2, R74.2: now also Q12.4 (G)
- net at D41.2 (A), R34.2, R40.2: now also Q5.4 (G)
- new net: C54.2, R54.2
- new net: C53.2, R53.2
- new net: C52.2, R52.2
Other:
- moved on the sheet: C46, C47, C48, C49, C50, C51, C56, C57, C58, C59, C60, C61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

Commit message: RS485Tx fix
Parts:
- removed J1: Conn_02x04_Counter_Clockwise, Button_Switch_THT:SW_DIP_SPSTx04_Slide_6.7x11.72mm_W7.62mm_P2.54mm_LowProfile, symbol Connector_Generic:Conn_02x04_Counter_Clockwise
- removed R7: 10k, Resistor_SMD:R_0603_1608Metric_Pad0.98x0.95mm_HandSolder, symbol Device:R
- added SW3: SW_DIP_x03, Button_Switch_THT:SW_DIP_SPSTx03_Slide_9.78x9.8mm_W7.62mm_P2.54mm, symbol Switch:SW_DIP_x03
- renumbered C84 to C82, C82 to C83, C83 to C84, J2 to J1, J11 to J10, J12 to J11, J3 to J2, J4 to J3, J5 to J4, J6 to J5, J7 to J6, J8 to J7, J9 to J8, J10 to J9, R11 to R10, R12 to R11, R13 to R12, R14 to R13, R15 to R14, R16 to R15, R17 to R16, R18 to R17, R19 to R18, R20 to R19, R21 to R20, R22 to R21, R23 to R22, R24 to R23, R25 to R24, R26 to R25, R27 to R26, R28 to R27, R29 to R28, R30 to R29, R31 to R30, R32 to R31, R33 to R32, R34 to R33, R35 to R34, R36 to R35, R37 to R36, R38 to R37, R39 to R38, R40 to R39, R41 to R40, R42 to R41, R43 to R42, R44 to R43, R45 to R44, R46 to R45, R47 to R46, R48 to R47, R49 to R48, R50 to R49, R51 to R50, R52 to R51, R53 to R52, R54 to R53, R55 to R54, R56 to R55, R57 to R56, R58 to R57, R59 to R58, R60 to R59, R61 to R60, R62 to R61, R63 to R62, R64 to R63, R65 to R64, R66 to R65, R67 to R66, R68 to R67, R69 to R68, R70 to R69, R8 to R7, R71 to R70, R72 to R71, R73 to R72, R74 to R73, R75 to R74, R76 to R75, R77 to R76, R78 to R77, R79 to R78, R80 to R79, R9 to R8, R81 to R80, R82 to R81, R83 to R82, R10 to R9, SW3 to SW4, SW4 to SW5, SW5 to SW6, SW6 to SW7, SW7 to SW8, SW8 to SW9
Connections:
- net +3V3: now also SW3.1, SW3.2, SW3.3
- net +5VD: no longer U23.2 (~{RE}), U23.3 (DE)
- net DIP_1: now also SW3.4
- net DIP_2: now also SW3.5
- net DIP_3: now also SW3.6
- net DIP_4 renamed RS485_DE
- net RS485_DE: now also U23.2 (~{RE}), U23.3 (DE)
Other:
- moved on the sheet: C82, R4, R5, R77

Commit message: beyond the MD10C Rev4.0
Parts:
- removed U13, U14, U15, U17, U18, U19: IRS2302S, Package_SO:SOIC-8_3.9x4.9mm_P1.27mm, symbol Driver_FET:IRS2302S
- added U13, U14, U15, U17, U18, U19: IR2184, Package_SO:SOIC-8_3.9x4.9mm_P1.27mm, symbol Driver_FET:IR2184
- Q1, Q10, Q11, Q12, Q2, Q3, Q4, Q5, Q6, Q7, Q8, Q9: value TPH4R008QM -> AGM028N08A; footprint MyLib:8-SOP Advance (5x5.75) -> Package_DFN_QFN:PQFN-8-EP_6x5mm_P1.27mm_Generic
- U1: value NJM7808SDL1 -> NJM7815SDL1
Connections:
- net GND: now also U13.3 (COM), U14.3 (COM), U15.3 (COM), U17.3 (COM), U18.3 (COM), U19.3 (COM)
- net Source_1A: now also U13.6 (VS)
- net Source_1B: now also U17.6 (VS)
- net Source_2A: now also U14.6 (VS)
- net Source_2B: now also U18.6 (VS)
- net Source_3A: now also U15.6 (VS)
- net Source_3B: now also U19.6 (VS)
- net at C71.2, C77.2, D57.1 (K)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: now also U19.8 (VB)
- net at C65.2, C73.2, D55.1 (K)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: now also U17.8 (VB)
- net at R76.2: now also U19.2 (~{SD})
- net at C36.2, C39.2, D33.1 (K)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: now also U15.8 (VB)
- net at D39.1 (K), R31.1: now also U14.7 (HO)
- net at C68.2, C75.2, D56.1 (K)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: now also U18.8 (VB)
- net at U21.4 (Y): now also U18.1 (IN)
- net at D53.1 (K), R72.1: now also U18.4 (LO)
- net at R75.2: now also U18.2 (~{SD})
- net at C34.2, C38.2, D29.1 (K)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: now also U14.8 (VB)
- net at D42.1 (K), R34.1: now also U15.4 (LO)
- net at U10.4 (Y): now also U13.1 (IN)
- net at R26.2: now also U13.2 (~{SD})
- net at D38.1 (K), R30.1: now also U13.4 (LO)
- net at D37.1 (K), R29.1: now also U13.7 (HO)
- net at C32.2, C37.2, D25.1 (K)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: now also U13.8 (VB)
- net at U20.4 (Y): now also U17.1 (IN)
- net at R74.2: now also U17.2 (~{SD})
- net at D52.1 (K), R71.1: now also U17.4 (LO)
- net at D49.1 (K), R68.1: now also U17.7 (HO)
- net at D40.1 (K), R32.1: now also U14.4 (LO)
- net at U12.4 (Y): now also U15.1 (IN)
- net at R28.2: now also U15.2 (~{SD})
- net at D41.1 (K), R33.1: now also U15.7 (HO)
- net at D50.1 (K), R69.1: now also U18.7 (HO)
- net at D51.1 (K), R70.1: now also U19.7 (HO)
- net at D54.1 (K), R73.1: now also U19.4 (LO)
- net at U22.4 (Y): now also U19.1 (IN)
- net at R27.2: now also U14.2 (~{SD})
- net at U11.4 (Y): now also U14.1 (IN)
- net +8V renamed +15V
- net +15V: now also U13.5 (VCC), U14.5 (VCC), U15.5 (VCC), U17.5 (VCC), U18.5 (VCC), U19.5 (VCC)
