File: MD_Stable.kicad_sch (KiCad schematic)
At the start: 298 parts, among them J1 XT30_Male, J10 Conn_01x08_Pin, J11 Conn_01x05_Socket, J2 XT60_Male, J3 RE1, J4 RE2, J5 RE3, J6 MO_XT60_Female1, J7 MO_XT60_Female2, J8 MO_XT60_Female3, J9 Conn_02x06_Odd_Even, Q1 AGM028N08A, Q10 AGM028N08A, Q11 AGM028N08A, Q12 AGM028N08A, Q2 AGM028N08A, Q3 AGM028N08A, Q4 AGM028N08A, Q5 AGM028N08A, Q6 AGM028N08A, Q7 AGM028N08A, Q8 AGM028N08A, Q9 AGM028N08A, SW1 SW_Push, SW2 SW_Push, SW3 SW_DIP_x03, SW4 PWM, SW5 PWM, SW6 PWM, SW7 DIR, SW8 DIR, SW9 DIR, U1 NJM7815SDL1, U10 74AHC1G08W5, U11 74AHC1G08W5, U12 74AHC1G08W5, U13 IR2184, U14 IR2184, U15 IR2184, U16 NE555D, U17 IR2184, U18 IR2184, U19 IR2184, U2 BA05CC0Tに似た何か, U20 74AHC1G08W5, U21 74AHC1G08W5, U22 74AHC1G08W5, U23 UTRS485G-S08-R, U24 UTRS485G-S08-R, U3 STM32G431K8Tx, U4 BA05CC0Tに似た何か, U5 BA033CC0FP, U6 π160M60, U7 74AHC1G04W5, U8 74AHC1G04W5, U9 74AHC1G04W5

Commit message: 時代はね、CANなんすよ
Parts:
- removed C82, C84: 0.1u, Capacitor_SMD:C_0603_1608Metric_Pad1.08x0.95mm_HandSolder, symbol Device:C
- removed J11: Conn_01x05_Socket, Connector_JST:JST_XH_S5B-XH-A-1_1x05_P2.50mm_Horizontal, symbol Connector:Conn_01x05_Socket
- removed R78: 120, Resistor_SMD:R_0603_1608Metric_Pad0.98x0.95mm_HandSolder, symbol Device:R
- removed R79, R80, R81, R82: 2.2k, Resistor_SMD:R_0603_1608Metric_Pad0.98x0.95mm_HandSolder, symbol Device:R
- removed U23, U24: UTRS485G-S08-R, Package_SO:SOP-8_3.76x4.96mm_P1.27mm, symbol Interface_UART:MAX3485
- added C1, C3: 22p, Capacitor_SMD:C_0603_1608Metric_Pad1.08x0.95mm_HandSolder, symbol Device:C
- added C83, C85: 0.1u, Capacitor_SMD:C_0603_1608Metric_Pad1.08x0.95mm_HandSolder, symbol Device:C
- added J11: FDCAN_1, Connector_JST:JST_XH_S2B-XH-A_1x02_P2.50mm_Horizontal, symbol Connector:Conn_01x02_Socket
- added U23: MCP2562-E-P, Package_SO:SOP-8_3.76x4.96mm_P1.27mm, symbol Interface_CAN_LIN:MCP2562-E-P
- added Y1: 8MHz, Crystal:Crystal_HC49-U_Vertical, symbol Device:Crystal
- renumbered C8 to C10, C9 to C11, C10 to C12, C11 to C13, C12 to C14, C13 to C15, C14 to C16, C15 to C17, C16 to C18, C17 to C19, C1 to C2, C18 to C20, C19 to C21, C20 to C22, C21 to C23, C22 to C24, C23 to C25, C24 to C26, C25 to C27, C26 to C28, C27 to C29, C28 to C30, C29 to C31, C30 to C32, C31 to C33, C32 to C34, C33 to C35, C34 to C36, C35 to C37, C36 to C38, C37 to C39, C2 to C4, C38 to C40, C39 to C41, C40 to C42, C41 to C43, C42 to C44, C43 to C45, C44 to C46, C45 to C47, C46 to C48, C47 to C49, C3 to C5, C48 to C50, C49 to C51, C50 to C52, C51 to C53, C52 to C54, C53 to C55, C54 to C56, C55 to C57, C56 to C58, C57 to C59, C4 to C6, C58 to C60, C59 to C61, C60 to C62, C61 to C63, C62 to C64, C63 to C65, C64 to C66, C65 to C67, C66 to C68, C67 to C69, C5 to C7, C68 to C70, C69 to C71, C70 to C72, C71 to C73, C72 to C74, C73 to C75, C74 to C76, C75 to C77, C76 to C78, C77 to C79, C6 to C8, C78 to C80, C79 to C81, C80 to C82, C81 to C84, C83 to C86, C7 to C9, D11 to D10, D9 to D11, D14 to D12, D12 to D13, D15 to D14, D13 to D15, D17 to D16, D18 to D17, D16 to D18, D4 to D3, D3 to D4, D10 to D9, R2 to R1, R12 to R11, R13 to R12, R11 to R13, R16 to R15, R17 to R16, R18 to R17, R19 to R18, R20 to R19, R1 to R2, R15 to R20, R22 to R21, R23 to R22, R24 to R23, R21 to R24, R4 to R3, R5 to R4, R6 to R5, R3 to R6, R9 to R7, R7 to R8, R8 to R9, SW3 to SW2, SW2 to SW3
Connections:
- net RS485_RX is gone; now on net RE1_B: U3.30 (PB7)
- net RS485_TX is gone; now on net RE1_A: U3.29 (PB6)
- net +3V3: now also C83.1, U23.5 (Vio)
- net +5VD: now also C85.1, U23.3 (VDD)
- net GNDD: now also C1.1, C3.1, C83.2, C85.2, U23.2 (VSS), U23.8 (STBY)
- net RE1_A: no longer U3.21 (PA11)
- net RE1_B: no longer U3.22 (PA12)
- net at R77.2: now also J11.2 (Pin_2), U23.6 (CANL)
- net at R77.1: now also J11.1 (Pin_1), U23.7 (CANH)
- net MCO_IN: no longer names the net of U3.2 (PF0)
- net MCO_IN: now also C1.2, Y1.1; no longer J9.10 (Pin_10)
- net RS485_DE: no longer names the net of U3.3 (PF1)
- net RS485_DE: now also C3.2, Y1.2
- new net FDCAN_RX: U23.4 (RXD), U3.21 (PA11)
- new net FDCAN_TX: U23.1 (TXD), U3.22 (PA12)
- no-connect marks 11 -> 10
Other:
- note added: "CAN"
- note removed: "RS-485"
- moved on the sheet: C21, D11, D13, D15, D18, D2, D4, R13, R2, R20, R24, R25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
